File: pcb/l130.kicad_sch (KiCad schematic)
At the start: 60 parts, among them CN1 Barrel_Jack, CN2 VGA, CN3 RJ45_Bel_SI-60062-F, CN4 Conn_02x05_Odd_Even, CN5 Conn_02x05_Odd_Even, CN6 AudioJack2_Dual_Switch, U1 AP1117-ADJ, U2 RTL8201CL, U3 EP1C6Q240C8N, U5 AT45DB041B, U6 K45643232H-UC60, U7 AP1117-33

Commit message: Update top photo without components, update list of components and schematic
Parts:
- added R? (x10): 2k, symbol Device:R
- added R?: 82, symbol Device:R
- OSC1: value 50 MHz? -> 80 MHz
Connections:
- net +3.3V: now also U?.18 (VCCIO), U?.3 (VCCIO), U?.34 (VCCIO), U?.39 (VCCINT), U?.51 (VCCIO), U?.66 (VCCIO), U?.82 (VCCIO), U?.91 (VCCINT), R?.2, R?.2, R?.2, R?.2, R?.2, R?.2, R?.2, R?.2, R?.2, R?.2
- net GND: now also U?.11 (GNDIO), U?.26 (GNDIO), U?.33 (GNDIO), U?.38 (GNDINT), U?.43 (GNDIO), U?.53 (GNDIO), U?.59 (GNDIO), U?.65 (GNDIO), U?.74 (GNDIO), U?.78 (GNDIO), U?.86 (GNDINT), U?.88 (OE1), U?.89 (GCLRn), U?.90 (OE2/GCLK2), U?.95 (GNDIO)
- net FAKE_TCK: now reaches CN4.1 (Pin_1)
- net FAKE_TCK: now also U?.57 (I/O), R?.1
- net FAKE_TDO: now reaches CN4.3 (Pin_3)
- net FAKE_TDO: now also U?.58 (I/O), R?.1
- net FAKE_TMS: now reaches CN4.5 (Pin_5)
- net FAKE_TMS: now also U?.60 (I/O), R?.1
- net FAKE_TDI: now reaches CN4.9 (Pin_9)
- net FAKE_TDI: now also U?.61 (I/O), R?.1
- net F_CONF_DONE: now reaches U?.16 (I/O)
- net C_SO: now reaches U?.21 (I/O)
- net C_SO: now also U5.8 (SO)
- net C_SI: now reaches U?.22 (I/O)
- net C_SI: now also U5.1 (SI)
- net C_SCK: now reaches U?.23 (I/O)
- net C_SCK: now also U5.2 (SCK)
- net C_NCS: now reaches U?.24 (I/O)
- net C_NCS: now also U5.4 (~{CS})
- net at U?.25 (I/O): now also R?.1
- net C_NRESET: now reaches U?.27 (I/O)
- net C_NRESET: now also U5.3 (~{RESET})
- net C_NWP: now reaches U?.28 (I/O)
- net C_NWP: now also U5.5 (~{WP})
- net F_97: now reaches U?.29 (I/O)
- net F_96: now reaches U?.30 (I/O)
- net F_95: now reaches U?.31 (I/O)
- net F_94: now reaches U?.32 (I/O)
- net at U?.36 (I/O): now also R?.1
- net F_88: now reaches U?.40 (I/O)
- net F_87: now reaches U?.41 (I/O)
- net F_86: now reaches U?.42 (I/O)
- net F_83: now reaches U?.44 (I/O)
- net F_81: now reaches U?.45 (I/O)
- net F_80: now reaches U?.46 (I/O)
- net F_79: now reaches U?.47 (I/O)
- net F_74: now reaches U?.49 (I/O)
- net F_73: now reaches U?.50 (I/O)
- net at U?.63 (I/O): now also R?.2
- net F_NCONFIG: now reaches U?.67 (I/O)
- net F_DATA0: now reaches U?.68 (I/O)
- net CY? renamed F_?
- removed net M?: U5.1 (SI), U5.2 (SCK), U5.3 (~{RESET}), U5.4 (~{CS}), U5.5 (~{WP}), U5.8 (SO)
- net M_CLK renamed C_CLK
- net TCK renamed C_TCK
- net C_TCK: now also CN5.1 (Pin_1), R?.1; no longer CN5.9 (Pin_9)
- net TDI renamed C_TDI
- net C_TDI: now also CN5.9 (Pin_9), R?.1; no longer CN5.1 (Pin_1)
- net TDO renamed C_TDO
- net C_TDO: now also CN5.3 (Pin_3), R?.1; no longer CN5.5 (Pin_5)
- net TMS renamed C_TMS
- net C_TMS: now also CN5.5 (Pin_5), R?.1; no longer CN5.3 (Pin_3)
- new net F_DCLK: R?.1
- no-connect marks 18 -> 62
Other:
- moved on the sheet: CN3, CN4, CN5, R?, U2
