File: pcb/l130.kicad_sch (KiCad schematic)
At the start: 71 parts, among them CN1 Barrel_Jack, CN2 VGA, CN3 RJ45_Bel_SI-60062-F, CN4 Conn_02x05_Odd_Even, CN5 Conn_02x05_Odd_Even, CN6 AudioJack2_Dual_Switch, U1 AP1117-ADJ, U2 RTL8201CL, U3 EP1C6Q240C8N, U5 AT45DB041B, U6 K45643232H-UC60, U7 AP1117-33

Commit message: Complete reverse engineering of board, update schematic
Connections:
- net F_73 is gone; now on net FC_73: U?.50 (I/O)
- net F_74 is gone; now on net FC_74: U?.49 (I/O)
- net F_79 is gone; now on net FC_79: U?.47 (I/O)
- net F_80 is gone; now on net FC_80: U?.46 (I/O)
- net F_81 is gone; now on net FC_81: U?.45 (I/O)
- net F_83 is gone; now on net FC_83: U?.44 (I/O)
- net F_86 is gone; now on net FC_86: U?.42 (I/O)
- net F_87 is gone; now on net FC_87: U?.41 (I/O)
- net F_88 is gone; now on net FC_88: U?.40 (I/O)
- net F_94 is gone; now on net FC_94: U?.32 (I/O)
- net F_95 is gone; now on net FC_95: U?.31 (I/O)
- net F_96 is gone; now on net FC_96: U?.30 (I/O)
- net +1V5: now also U3.110 (VCCINT), U3.154 (VCCA_PLL2), U3.191 (VCCINT), U3.211 (VCCINT), U3.229 (VCCINT), U3.27 (VCCA_PLL1), U3.72 (VCCINT), U3.90 (VCCINT)
- net +3.3V: now also U3.112 (VCCIO4), U3.130 (VCCIO3), U3.157 (VCCIO3), U3.172 (VCCIO3), U3.189 (VCCIO2), U3.209 (VCCIO2), U3.22 (VCCIO1), U3.231 (VCCIO2), U3.34 (MSEL0), U3.51 (VCCIO1), U3.70 (VCCIO4), U3.9 (VCCIO1), U3.92 (VCCIO4)
- net F_CONF_DONE: now also U3.145 (CONF_DONE)
- net F_DATA0: now also U3.25 (DATA0)
- net F_DCLK: now also U3.36 (DCLK)
- net F_NCONFIG: now also U3.26 (nCONFIG)
- net GND: now also U3.10 (GND), U3.109 (GND), U3.111 (GND), U3.129 (GND), U3.142 (GND), U3.150 (GNDG_PLL2), U3.151 (GNDA_PLL2), U3.171 (GND), U3.190 (GND), U3.192 (GND), U3.210 (GND), U3.212 (GND), U3.230 (GND), U3.232 (GND), U3.234 (I/O), U3.236 (I/O), U3.237 (I/O), U3.238 (I/O), U3.30 (GNDA_PLL1), U3.31 (GNDG_PLL1), U3.33 (nCE), U3.35 (MSEL1), U3.40 (GND), U3.52 (GND), U3.69 (GND), U3.71 (GND), U3.89 (GND), U3.91 (GND)
- net AUDIO_1: now reaches U3.1 (I/O)
- net AUDIO_1: now also CN6.S1
- net RESETB: now reaches U3.100 (I/O)
- net RESETB: now also R?.1
- net X1: now reaches U3.101 (I/O)
- net X1: now also R?.1
- net DQ15: now reaches U3.102 (I/O)
- net DQ15: now also U6.85 (DQ15)
- net DQ14: now reaches U3.103 (I/O)
- net DQ14: now also U6.83 (DQ14)
- net DQ13: now reaches U3.104 (I/O)
- net DQ13: now also U6.82 (DQ13)
- net DQ12: now reaches U3.105 (I/O)
- net DQ12: now also U6.80 (DQ12)
- net DQ11: now reaches U3.106 (I/O)
- net DQ11: now also U6.79 (DQ11)
- net DQ10: now reaches U3.107 (I/O)
- net DQ10: now also U6.77 (DQ10)
- net DQ9: now reaches U3.108 (I/O)
- net DQ9: now also U6.76 (DQ9)
- net DQ8: now reaches U3.113 (I/O)
- net DQ8: now also U6.74 (DQ8)
- net DQM1: now reaches U3.114 (I/O)
- net DQM1: now also U6.71 (DQM1)
- net CLK: now reaches U3.115 (I/O)
- net CLK: now also R?.2
- net A9: now reaches U3.116 (I/O)
- net A9: now also U6.66 (A9)
- net A5: now reaches U3.117 (I/O)
- net A5: now also U6.62 (A5)
- net A6: now reaches U3.118 (I/O)
- net A6: now also U6.63 (A6)
- net A8: now reaches U3.119 (I/O)
- net A8: now also U6.65 (A8)
- net A7: now reaches U3.120 (I/O)
- net A7: now also U6.64 (A7)
- net A4: now reaches U3.121 (I/O)
- net A4: now also U6.61 (A4)
- net A3: now reaches U3.122 (I/O)
- net A3: now also U6.60 (A3)
- net DQM3: now reaches U3.123 (I/O)
- net DQ31: now reaches U3.124 (I/O)
- net DQ31: now also U6.56 (DQ31)
- net DQ30: now reaches U3.125 (I/O)
- net DQ30: now also U6.54 (DQ30)
- net DQ29: now reaches U3.126 (I/O)
- net DQ29: now also U6.53 (DQ29)
- net DQ28: now reaches U3.127 (I/O)
- net DQ28: now also U6.51 (DQ28)
- net DQ27: now reaches U3.128 (I/O)
- net DQ27: now also U6.50 (DQ27)
- net DQ26: now reaches U3.131 (I/O)
- net DQ26: now also U6.48 (DQ26)
- net DQ25: now reaches U3.132 (I/O)
- net DQ25: now also U6.47 (DQ25)
- net DQ24: now reaches U3.133 (I/O)
- net DQ24: now also U6.45 (DQ24)
- net TXD2: now reaches U3.134 (I/O)
- net TXD2: now also U2.4 (TXD2)
- net TXD1: now reaches U3.135 (I/O)
- net TXD1: now also U2.5 (TXD1)
- net TXD0: now reaches U3.136 (I/O)
- net TXD0: now also U2.6 (TXD0)
- net TXC: now reaches U3.137 (I/O)
- net TXC: now also R?.1
- net RXC: now reaches U3.138 (I/O)
- net RXC: now also R?.2
- net RXD3: now reaches U3.139 (I/O)
- net RXD3: now also U2.18 (RXD3)
- net RXD2: now reaches U3.140 (I/O)
- net RXD2: now also U2.19 (RXD2)
- net RXD1: now reaches U3.141 (I/O)
- net RXD1: now also U2.20 (RXD1)
- net RXD0: now reaches U3.143 (I/O)
- net RXD0: now also U2.21 (RXD0)
- net RXDV: now reaches U3.144 (I/O)
- net RXDV: now also U2.22 (RXDV)
- net F_CLK: now reaches U3.153 (CLK2)
- net F_CLK: now also R?.1, U3.28 (CLK0)
- net CRS: now reaches U3.156 (I/O)
- net CRS: now also U2.23 (CRS)
- net DQ23: now reaches U3.158 (I/O)
- net DQ23: now also U6.42 (DQ23)
- net DQ22: now reaches U3.159 (I/O)
- net DQ22: now also U6.40 (DQ22)
- net DQ21: now reaches U3.160 (I/O)
- net DQ21: now also U6.39 (DQ21)
- net DQ20: now reaches U3.161 (I/O)
- net DQ20: now also U6.37 (DQ20)
- net DQ19: now reaches U3.162 (I/O)
- net DQ19: now also U6.36 (DQ19)
- net DQ17: now reaches U3.164 (I/O)
- net DQ17: now also U6.33 (DQ17)
- net DQ16: now reaches U3.165 (I/O)
- net DQ16: now also U6.31 (DQ16)
- net VGA_B0: now reaches U3.166 (I/O)
- net VGA_B0: now also RN?.4 (R4.1)
- net VGA_B1: now reaches U3.167 (I/O)
- net VGA_B1: now also RN?.3 (R3.1)
- net VGA_B2: now reaches U3.168 (I/O)
- net VGA_B2: now also RN?.2 (R2.1)
- net VGA_B4: now reaches U3.169 (I/O)
- net VGA_B4: now also RN?.3 (R3.1)
- net VGA_B3: now reaches U3.170 (I/O)
- net VGA_B3: now also RN?.4 (R4.1)
- net DQM2: now reaches U3.173 (I/O)
- net DQM2: now also U6.28 (DQM2), U6.59 (DQM3)
- net A2: now reaches U3.174 (I/O)
- net A2: now also U6.27 (A2)
- net A1: now reaches U3.175 (I/O)
- net A1: now also U6.26 (A1)
- net A0: now reaches U3.176 (I/O)
- net A0: now also U6.25 (A0)
- net A10: now reaches U3.177 (I/O)
- net A10: now also U6.24 (A10)
- net BA1: now reaches U3.178 (I/O)
- net BA1: now also U6.23 (BA1)
- net BA0: now reaches U3.179 (I/O)
- net BA0: now also U6.22 (BA0)
- net FXER_FXEN: now reaches U3.180 (I/O)
- net NWE: now reaches U3.181 (I/O)
- net NWE: now also U6.17 (~{WE})
- net NCAS: now reaches U3.182 (I/O)
- net NCAS: now also U6.18 (~{CAS})
- net NRAS: now reaches U3.183 (I/O)
- net NRAS: now also U6.19 (~{RAS})
- net NCS: now reaches U3.184 (I/O)
- net NCS: now also U6.20 (~{CS})
- net DQM0: now reaches U3.185 (I/O)
- net DQM0: now also U6.16 (DQM0)
- net DQ7: now reaches U3.186 (I/O)
- net DQ7: now also U6.13 (DQ7)
- net DQ6: now reaches U3.187 (I/O)
- net DQ6: now also U6.11 (DQ6)
- net DQ5: now reaches U3.188 (I/O)
- net DQ5: now also U6.10 (DQ5)
- net DQ4: now reaches U3.193 (I/O)
- net DQ4: now also U6.8 (DQ4)
- net DQ3: now reaches U3.194 (I/O)
- net DQ3: now also U6.7 (DQ3)
- net DQ2: now reaches U3.195 (I/O)
- net DQ2: now also U6.5 (DQ2)
- net DQ1: now reaches U3.196 (I/O)
- net DQ1: now also U6.4 (DQ1)
- net DQ0: now reaches U3.197 (I/O)
- net DQ0: now also U6.2 (DQ0)
- net TXD3: now reaches U3.198 (I/O)
- net TXD3: now also U2.3 (TXD3)
- net TXEN: now reaches U3.199 (I/O)
- net TXEN: now also U2.2 (TXEN)
- net AUDIO_2: now reaches U3.2 (I/O)
- net AUDIO_2: now also CN6.T1
- net COL: now reaches U3.200 (I/O)
- net COL: now also U2.1 (COL)
- net MDC: now reaches U3.201 (I/O)
- net MDC: now also U2.25 (MDC)
- net MDIO: now reaches U3.202 (I/O)
- net MDIO: now also U2.26 (MDIO)
- net MOUSE_DATA: now reaches U3.203 (I/O)
- net MOUSE_DATA: now also J?.1
- net MOUSE_CLK: now reaches U3.204 (I/O)
- net MOUSE_CLK: now also J?.5
- net KBD_CLK: now reaches U3.205 (I/O)
- net KBD_CLK: now also J?.5
- net KBD_DATA: now reaches U3.206 (I/O)
- net KBD_DATA: now also J?.1
- net VGA_R4: now reaches U3.217 (I/O)
- net VGA_R4: now also RN?.3 (R3.1)
- net VGA_R3: now reaches U3.220 (I/O)
- net VGA_R3: now also RN?.4 (R4.1)
- net VGA_R2: now reaches U3.221 (I/O)
- net VGA_R2: now also RN?.2 (R2.1)
- net VGA_R1: now reaches U3.222 (I/O)
- net VGA_R1: now also RN?.3 (R3.1)
- net VGA_R0: now reaches U3.223 (I/O)
- net VGA_R0: now also RN?.4 (R4.1)
- net VGA_G5: now reaches U3.224 (I/O)
- net VGA_G5: now also RN?.2 (R2.1)
- net VGA_G4: now reaches U3.225 (I/O)
- net VGA_G4: now also RN?.3 (R3.1)
- net VGA_G3: now reaches U3.226 (I/O)
- net VGA_G3: now also RN?.4 (R4.1)
- net VGA_G2: now reaches U3.227 (I/O)
- net VGA_G2: now also RN?.2 (R2.1)
- net VGA_G1: now reaches U3.228 (I/O)
- net VGA_G1: now also RN?.3 (R3.1)
- net VGA_G0: now reaches U3.233 (I/O)
- net VGA_G0: now also RN?.4 (R4.1)
- net FC_73: now reaches U3.73 (I/O)
- net FC_74: now reaches U3.74 (I/O)
- net FC_79: now reaches U3.79 (I/O)
- net FC_80: now reaches U3.80 (I/O)
- net FC_81: now reaches U3.81 (I/O)
- net FC_83: now reaches U3.83 (I/O)
- net LED3: now reaches U3.85 (I/O)
- net LED3: now also D?.2 (A)
- net FC_86: now reaches U3.86 (I/O)
- net FC_87: now reaches U3.87 (I/O)
- net FC_88: now reaches U3.88 (I/O)
- net LED2: now reaches U3.93 (I/O)
- net LED2: now also D?.2 (A)
- net FC_94: now reaches U3.94 (I/O)
- net FC_95: now reaches U3.95 (I/O)
- net FC_96: now reaches U3.96 (I/O)
- net F_97 renamed FC_97
- removed net F_?: CN2.13, CN2.14, CN6.S1, CN6.T1, D?.2 (A), D?.2 (A), J?.1, J?.1, J?.5, J?.5, R?.1, R?.1, R?.1, R?.1, R?.2, R?.2, RN?.2 (R2.1), RN?.2 (R2.1), RN?.2 (R2.1), RN?.2 (R2.1), RN?.3 (R3.1), RN?.3 (R3.1), RN?.3 (R3.1), RN?.3 (R3.1), RN?.3 (R3.1), RN?.3 (R3.1), RN?.4 (R4.1), RN?.4 (R4.1), RN?.4 (R4.1), RN?.4 (R4.1), RN?.4 (R4.1), RN?.4 (R4.1), U2.1 (COL), U2.18 (RXD3), U2.19 (RXD2), U2.2 (TXEN), U2.20 (RXD1), U2.21 (RXD0), U2.22 (RXDV), U2.23 (CRS), U2.24 (RXER/FXEN), U2.25 (MDC), U2.26 (MDIO), U2.3 (TXD3), U2.4 (TXD2), U2.5 (TXD1), U2.6 (TXD0), U6.10 (DQ5), U6.11 (DQ6), U6.13 (DQ7), U6.16 (DQM0), U6.17 (~{WE}), U6.18 (~{CAS}), U6.19 (~{RAS}), U6.2 (DQ0), U6.20 (~{CS}), U6.21 (A11), U6.22 (BA0), U6.23 (BA1), U6.24 (A10), U6.25 (A0), U6.26 (A1), U6.27 (A2), U6.28 (DQM2), U6.31 (DQ16), U6.33 (DQ17), U6.34 (DQ18), U6.36 (DQ19), U6.37 (DQ20), U6.39 (DQ21), U6.4 (DQ1), U6.40 (DQ22), U6.42 (DQ23), U6.45 (DQ24), U6.47 (DQ25), U6.48 (DQ26), U6.5 (DQ2), U6.50 (DQ27), U6.51 (DQ28), U6.53 (DQ29), U6.54 (DQ30), U6.56 (DQ31), U6.59 (DQM3), U6.60 (A3), U6.61 (A4), U6.62 (A5), U6.63 (A6), U6.64 (A7), U6.65 (A8), U6.66 (A9), U6.7 (DQ3), U6.71 (DQM1), U6.74 (DQ8), U6.76 (DQ9), U6.77 (DQ10), U6.79 (DQ11), U6.8 (DQ4), U6.80 (DQ12), U6.82 (DQ13), U6.83 (DQ14), U6.85 (DQ15)
- new net DQ18: U6.34 (DQ18)
- new net RXER_FXEN: U2.24 (RXER/FXEN)
- new net VGA_HS: CN2.13
- new net VGA_VS: CN2.14
- no-connect marks 62 -> 136
